File: flex-cv-in/_autosave-biased-CV-input-unity.kicad_sch (KiCad schematic)
At the start: 20 parts, among them J1 3.5mm_Mono_Switched, J2 Conn_01x04, U1 TLV9061xDBV

Commit message: Rename and update flex-cv-in
Parts:
- removed JP1: NORMAL_HIGH, Jumper:SolderJumper-2_P1.3mm_Open_RoundedPad1.0x1.5mm, symbol Jumper:SolderJumper_2_Open
- removed JP2: NORMAL_LOW, Jumper:SolderJumper-2_P1.3mm_Open_RoundedPad1.0x1.5mm, symbol Jumper:SolderJumper_2_Open
- removed JP3: JACK_DETECT, Jumper:SolderJumper-2_P1.3mm_Open_RoundedPad1.0x1.5mm, symbol Jumper:SolderJumper_2_Open
- added JP6: RIN_CUT, Jumper:SolderJumper-2_P1.3mm_Bridged_RoundedPad1.0x1.5mm, symbol Jumper:SolderJumper_2_Bridged
- added R7: 10k, Resistor_SMD:R_0805_2012Metric, symbol Device:R_US
- J2: value Conn_01x04 -> HDR
- JP4: value SolderJumper_3_Open -> POT_1; footprint Jumper:SolderJumper-3_P1.3mm_Open_RoundedPad1.0x1.5mm -> elemental_jumper:SolderJumper-3_P1.3mm_Open_RoundedPad1.0x1.5mm
- JP5: value SolderJumper_3_Open -> POT_3; footprint Jumper:SolderJumper-3_P1.3mm_Open_RoundedPad1.0x1.5mm -> elemental_jumper:SolderJumper-3_P1.3mm_Open_RoundedPad1.0x1.5mm
Connections:
- net JACK_NORMAL is gone; now on net JACK_DETECT: J1.3 (SW)
- net +3.3V: no longer JP5.1 (A)
- net CV_IN: now also JP5.1 (A), JP6.2 (B), R7.2; no longer R2.1
- net CV_OUT: now also J2.2 (Pin_2); no longer J2.3 (Pin_3)
- net GND: now also J2.3 (Pin_3), R7.1; no longer J2.4 (Pin_4), JP4.1 (A)
- net JACK_DETECT: now also J2.4 (Pin_4); no longer J2.2 (Pin_2)
- net VREF_1.65V: now also JP4.1 (A)
- new net R_IN: JP6.1 (A), R2.1
Other:
- note added: "Bridge 2+3 to bias incoming CV Bridge 1+2 (and cut JP6) to attenuate incoming CV"
- note removed: "Bridge 1+2 or 2+3 to flip potentiometer direction without cutting traces or rewiring."
- moved on the sheet: C1, C2, C3, C4, D1, J1, J2, JP4, JP5, R1, R2, R3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
