File: mixer-4ch-mono/mixer-main/mixer-main.kicad_sch (KiCad schematic)
At the start: 28 parts, among them J1 USB_C_Receptacle_PowerOnly_6P, J3 Conn_01x08, J6 Conn_01x02, U1 TLV9062IDR, U2 TLV431AIDBZR, U3 SPX3819M5-L-3-3

Commit message: Update mixer-main
Continued with layout.
Parts:
- removed J6: Conn_01x02, Connector_PinSocket_2.54mm:PinSocket_1x02_P2.54mm_Vertical, symbol Connector_Generic:Conn_01x02
- removed RV1: A/B10k, Connector_PinSocket_2.54mm:PinSocket_1x03_P2.54mm_Vertical, symbol Device:R_Potentiometer_US
- added J2: HEADER_OUT, Connector_PinHeader_2.54mm:PinHeader_1x04_P2.54mm_Vertical, symbol Connector_Generic:Conn_01x04
- added TP1: VREF, TestPoint:TestPoint_THTPad_D2.0mm_Drill1.0mm, symbol Connector:TestPoint
- added TP2: 3.3V, TestPoint:TestPoint_THTPad_D2.0mm_Drill1.0mm, symbol Connector:TestPoint
- added TP3: VBUS, TestPoint:TestPoint_THTPad_D2.0mm_Drill1.0mm, symbol Connector:TestPoint
- added TP4: MIX_NODE, TestPoint:TestPoint_THTPad_D2.0mm_Drill1.0mm, symbol Connector:TestPoint
- C6: footprint Capacitor_SMD:C_0603_1608Metric -> Capacitor_SMD:C_0805_2012Metric
- J3: footprint (none) -> Connector_PinHeader_2.54mm:PinHeader_1x08_P2.54mm_Vertical
Connections:
- net VREF_1.65 is gone; now on net VREF_1.65V: J3.2 (Pin_2), J3.4 (Pin_4), J3.6 (Pin_6), J3.8 (Pin_8)
- net +3.3V: now also TP2.1
- net GND: now also J2.2 (Pin_2)
- net IN_SIG_2: now also J3.3 (Pin_3); no longer J3.5 (Pin_5)
- net IN_SIG_3: now also J3.5 (Pin_5); no longer J3.3 (Pin_3)
- net VREF_1.65V: now also TP1.1
- net at R1.1, R10.2, R7.2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: now also TP4.1
- net TO_OPAMP_7: now reaches R11.1, U1.7
- net TO_OPAMP_7: now also J2.3 (Pin_3)
- net MIX_OUT: now reaches C7.1, JP1.1 (A)
- net MIX_OUT: now also J2.1 (Pin_1)
- net LDO_IN: now reaches C4.1, FB1.2, U3.1 (IN), U3.3 (EN)
- net LDO_FB: now reaches C6.1, U3.4 (BP)
- net at FB1.1, J1.A9 (VBUS), J1.B9 (VBUS): now also TP3.1
- net TO_OPAMP_6: now reaches R2.2, U1.6 (-)
- net TO_OPAMP_6: now also J2.4 (Pin_4)
- no-connect marks 1 -> 0
Other:
- note added: "bus gain potentiometer (off board)"
- note added: "channel gain potentiometers (off board)"
- note removed: "bus gain potentiometer"
- note removed: "channel gain potentiometers"
- moved on the sheet: C7, JP1, R11
