File: mixer-4ch-mono/mixer-chan/mixer-chan.kicad_pcb (KiCad board)
At the start: 2 copper layers, 30 x 17 mm, 3 parts, among them J1 3.5mm_Mono_Switched, J2 Conn_01x03

Commit message: Finalize mixer-4ch-mono rev. A
Other:
- board text added: "gnd"
- board text added: "mixer-chan"
- board text added: "out"
- board text added: "patch_bits"
- board text added: "rev A"
- board text added: "vref"
- board text removed: "GND"
- board text removed: "SIG"
- board text removed: "VREF"
