File: mixer-4ch-mono/mixer-out/mixer-out.kicad_pcb (KiCad board)
At the start: 2 copper layers, 30 x 17 mm, 3 parts, among them J1 3.5mm_Mono_Switched, J3 Conn_01x04

Commit message: Finalize mixer-4ch-mono rev. A
Parts:
- RV1: value A/B10k -> a/b10k
Other:
- board text added: "3.5mm mono"
- board text added: "gnd"
- board text added: "mixer-out"
- board text added: "op6"
- board text added: "op7"
- board text added: "out"
- board text added: "patch_bits"
- board text added: "rev A"
- board text added: "rk097n"
- board text added: "switched"
- board text removed: "3.5mm Mono"
- board text removed: "GND"
- board text removed: "OUT"
- board text removed: "RK097N"
- board text removed: "Switched"
- board text removed: "TO6"
- board text removed: "TO7"
